File: kicad/arduino_led_tester_cover/arduino_led_tester_cover.kicad_pcb (KiCad board)
At the start: 2 copper layers, 50 x 80 mm, 12 parts

Commit message: updates to cover pcb and fabrication files
Routing:
- removed copper zone on F.Cu, net (none)
Changed lines of the file:
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@@
 		(net 0)
-	)
-	(zone
-		(net 0)
-		(net_name "")
-		(layer "F.Cu")
-		(hatch edge 0.5)
-		(connect_pads
-			(clearance 0.1)
-		)
-		(min_thickness 0.25)
-		(filled_areas_thickness no)
-		(fill yes
-			(thermal_gap 0.5)
-			(thermal_bridge_width 0.5)
-			(island_removal_mode 1)
-			(island_area_min 10)
-		)
-		(polygon
-			(pts
-				(xy 25.095 70.605) (xy 47.945 70.605) (xy 47.945 92.005) (xy 25.095 92.005)
-			)
-		)
 	)
 	(group ""
